File: CD2003-IQ-v4/BoB.kicad_sch (KiCad schematic)
At the start: 43 parts, among them J1 ANTENNA, U1 CD2003GB_GP, U2 CD2003GB_GP, U3 ADP-2-1W+, U4 SI5351_Module

Commit message: In-flight projects and ideas
Parts:
- removed D1, D2, D7, D8: 1N4148, Diode_SMD:D_SOD-323_HandSoldering, symbol Device:D
- removed J1: ANTENNA, Connector_Coaxial:SMA_Samtec_SMA-J-P-X-ST-EM1_EdgeMount, symbol Connector:Conn_Coaxial
- removed TP1: TestPoint, symbol Connector:TestPoint
- removed U3: ADP-2-1W+, footprints:MC-CDXXX-Modded, symbol ADP-2-1W_:ADP-2-1W+
- added ACLK1: ACLK, TestPoint:TestPoint_Pad_4.0x4.0mm, symbol Connector_Generic:Conn_01x01
- added D3, D4, D5, D6: 1N4148, Diode_SMD:D_SOD-123, symbol Device:D
- added GND1: GND, TestPoint:TestPoint_Pad_4.0x4.0mm, symbol Connector_Generic:Conn_01x01
- added I1: I, TestPoint:TestPoint_Pad_4.0x4.0mm, symbol Connector_Generic:Conn_01x01
- added J2, J3: ANTENNA, Connector_Coaxial:SMA_Samtec_SMA-J-P-X-ST-EM1_EdgeMount, symbol Connector:Conn_Coaxial
- added Q1: Q, TestPoint:TestPoint_Pad_4.0x4.0mm, symbol Connector_Generic:Conn_01x01
- added SCL1: SCL, TestPoint:TestPoint_Pad_4.0x4.0mm, symbol Connector_Generic:Conn_01x01
- added SDA1: SDA, TestPoint:TestPoint_Pad_4.0x4.0mm, symbol Connector_Generic:Conn_01x01
- C19, C2: value 10uF -> 10u
Connections:
- net +5V: no longer U4.1 (VIN)
- net 5VCLEAN: now also U4.1 (VIN)
- net GND: now also D3.2 (A), D4.1 (K), D5.2 (A), D6.1 (K), GND1.1 (Pin_1), J2.2 (Ext), J3.2 (Ext)
- net I: now also I1.1 (Pin_1)
- net Q: now also Q1.1 (Pin_1)
- net SCL: now also SCL1.1 (Pin_1)
- net SDA: now also SDA1.1 (Pin_1)
- net at C14.2: now also D5.1 (K), D6.2 (A), J3.1 (In)
- net at C17.2: now also D3.1 (K), D4.2 (A), J2.1 (In)
- net ACLK: now reaches U4.5 (S2)
- net ACLK: now also ACLK1.1 (Pin_1)
- no-connect marks 11 -> 10
