File: ADE-1+-BoB/Mixer.kicad_pcb (KiCad board)
At the start: 2 copper layers, 26.2 x 25.8 mm, 8 parts

Commit message: pHAT
Parts:
- MX1: value ADE-1 -> ADE-1+
- SMA1, SMA2, SMA3: footprint footprints:SMA_EDGELAUNCH_Modded -> Connector_Coaxial:SMA_Samtec_SMA-J-P-X-ST-EM1_EdgeMount
- moved SMA1 2.09 mm to (88.0, 105.6), turned to -90 degrees
- moved SMA3 1.62 mm to (108.9, 105.7), turned to 90 degrees
- moved SMA2 1.42 mm to (98.6, 116.7), turned to 0 degrees
