File: ADE-1+-BoB/Mixer.kicad_sch (KiCad schematic)
At the start: 8 parts

Commit message: pHAT
Parts:
- BNC1: footprint footprints:SMA_EDGELAUNCH_Modded -> Connector_Coaxial:SMA_Samtec_SMA-J-P-X-ST-EM1_EdgeMount
Changed lines of the file:
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@@
       (effects (font (size 1.27 1.27)) hide)
     )
-    (property "Footprint" "footprints:SMA_EDGELAUNCH_Modded" (at 59.69 50.8 0)
+    (property "Footprint" "Connector_Coaxial:SMA_Samtec_SMA-J-P-X-ST-EM1_EdgeMount" (at 59.69 50.8 0)
       (effects (font (size 1.27 1.27)) hide)
     )
@@
       (effects (font (size 1.27 1.27)) hide)
     )
-    (property "Footprint" "footprints:SMA_EDGELAUNCH_Modded" (at 90.17 50.8 0)
+    (property "Footprint" "Connector_Coaxial:SMA_Samtec_SMA-J-P-X-ST-EM1_EdgeMount" (at 90.17 50.8 0)
       (effects (font (size 1.27 1.27)) hide)
     )
@@
       (effects (font (size 1.27 1.27)) hide)
     )
-    (property "Footprint" "footprints:SMA_EDGELAUNCH_Modded" (at 74.93 35.56 0)
-      (effects (font (size 1.27 1.27)) hide)
-    )
+    (property "Footprint" "Connector_Coaxial:SMA_Samtec_SMA-J-P-X-ST-EM1_EdgeMount" (at 74.93 35.56 0)
+      (effects (font (size 1.27 1.27)) hide)
+    )
